Commit message: Updated fake_lidar_with_tf, generate_luts Changes to be committed: 	modified:   src/fake_lidar_with_tf/fake_lidar_with_tf/fake_lidar_with_tf.py 	modified:   src/freespace_detection/freespace_detection/floor_detector.py 	modified:   src/freespace_detection/scripts/distance_lut.npy 	modified:   src/freespace_detection/scripts/generate_luts.py 	modified:   src/omo_r1_description/urdf/omo_r1.urdf 	modified:   src/omo_r1_navigation2/param/omo_r1.yaml

File: src/omo_r1_description/urdf/omo_r1.urdf (robot description, URDF)
Before this commit: robot omo_r1, 8 links, 7 joints
Links:
- added link camera_link
Joints:
- added joint camera_joint: type fixed, parent base_link, child camera_link, origin xyz=-0.5 0 0.2 rpy=0 0 0
